File: pcb/MacRoPadv2.kicad_pcb (KiCad board)
At the start: 2 copper layers, 90 x 66 mm, 15 parts, among them J1 Conn_01x04, SW1 SW_Push, SW2 SW_Push, SW3 SW_Push, SW4 SW_Push, SW5 SW_Push, SW6 SW_Push, SW7 RotaryEncoder, SW8 RotaryEncoder, U1 MOUDLE-SEEEDUINO-XIAO

Commit message: Add files via upload
Parts:
- added REF**: MountingHole_3.2mm_M3, MountingHole:MountingHole_3.2mm_M3, F.Cu at (187.6, 88.2)
Other:
- board text added: "m3 3.2mm"
Changed lines of the file:
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@@
 			(drillshape 0)
 			(scaleselection 1)
-			(outputdirectory "gerber file macRo pad/")
+			(outputdirectory "gerber/")
 		)
 	)
@@
 		)
 	)
+	(footprint "MountingHole:MountingHole_3.2mm_M3"
+		(layer "F.Cu")
+		(at 187.6 88.2)
+		(descr "Mounting Hole 3.2mm, M3, no annular, generated by kicad-footprint-generator mountinghole.py")
+		(tags "mountinghole M3")
+		(property "Reference" "REF**"
+			(at 0 -4.15 0)
+			(layer "F.SilkS")
+			(hide yes)
+			(effects
+				(font
+					(size 1 1)
+					(thickness 0.15)
+				)
+			)
+		)
+		(property "Value" "MountingHole_3.2mm_M3"
+			(at 0 4.15 0)
+			(layer "F.Fab")
+			(hide yes)
+			(effects
+				(font
+					(size 1 1)
+					(thickness 0.15)
+				)
+			)
+		)
+		(property "Datasheet" ""
+			(at 0 0 0)
+			(layer "F.Fab")
+			(hide yes)
+			(effects
+				(font
+					(size 1.27 1.27)
+					(thickness 0.15)
+				)
+			)
+		)
+		(property "Description" ""
+			(at 0 0 0)
+			(layer "F.Fab")
+			(hide yes)
+			(effects
+				(font
+					(size 1.27 1.27)
+					(thickness 0.15)
+				)
+			)
+		)
+		(attr exclude_from_pos_files exclude_from_bom)
+		(fp_circle
+			(center 0 0)
+			(end 3.2 0)
+			(stroke
+				(width 0.15)
+				(type solid)
+			)
+			(fill no)
+			(layer "Cmts.User")
+		)
+		(fp_circle
+			(center 0 0)
+			(end 3.45 0)
+			(stroke
+				(width 0.05)
+				(type solid)
+			)
+			(fill no)
+			(layer "F.CrtYd")
+		)
+		(pad "" np_thru_hole circle
+			(at 0 0)
+			(size 3.2 3.2)
+			(drill 3.2)
+			(layers "*.Cu" "*.Mask")
+		)
+		(embedded_fonts no)
+	)
 	(footprint "footprints:XIAO-RP2040-DIP"
 		(layer "B.Cu")
@@
 		(layer "Edge.Cuts")
 	)
+	(gr_text "m3 3.2mm"
+		(at 183.7 93.3 0)
+		(layer "F.SilkS")
+		(effects
+			(font
+				(size 1 1)
+				(thickness 0.2)
+				(bold yes)
+			)
+			(justify left bottom)
+		)
+	)
 	(gr_text "MacRo Pad"

Commit message: Add files via upload
Parts:
- added D6: 1N4148, Diode_THT:D_DO-35_SOD27_P7.62mm_Horizontal, B.Cu at (152.5, 51.6)
- D1, D2, D3, D4, D5: moved to B.Cu
- moved D2 8.10 mm to (152.5, 59.4), turned to 0 degrees
- moved D3 7.84 mm to (152.5, 56.8), turned to 0 degrees
- moved D4 7.53 mm to (152.5, 62.0), turned to 0 degrees
- moved D5 7.53 mm to (152.5, 64.6), turned to 0 degrees
- moved D1 7.51 mm to (152.5, 54.2), turned to 0 degrees
Connections:
- net /SCL renamed pin 3 display
- net /SDA renamed pin 4 display
- net Net-(U1-PA5_A9_D9_MISO) renamed SW8 A
- net Net-(U1-PA6_A10_D10_MOSI) renamed SW8 B
- net Net-(U1-PA7_A8_D8_SCK) renamed SW7 B
- net Net-(U1-PB09_A7_D7_RX) renamed SW7 A
- D1 pad 1: Net-(D1-K) -> row 1
- D2 pad 1: Net-(D2-K) -> row 2
- D3 pad 1: Net-(D3-K) -> row 1
- D4 pad 1: Net-(D4-K) -> row 2
- D5 pad 1: Net-(D5-K) -> row 2
- SW1 pad 1: Net-(D1-K) -> Net-(D1-A)
- SW1 pad 2: Net-(D3-K) -> column 1
- SW2 pad 1: Net-(D2-K) -> Net-(D2-A)
- SW2 pad 2: Net-(D3-K) -> column 1
- SW3 pad 1: Net-(D1-K) -> Net-(D3-A)
- SW3 pad 2: Net-(D4-K) -> column 2
- SW4 pad 1: Net-(D2-K) -> Net-(D4-A)
- SW4 pad 2: Net-(D4-K) -> column 2
- SW5 pad 1: Net-(D1-K) -> Net-(D6-A)
- SW5 pad 2: Net-(D5-K) -> column 3
- SW6 pad 1: Net-(D2-K) -> Net-(D5-A)
- SW6 pad 2: Net-(D5-K) -> column 3
- U1 pad 1: Net-(D1-A) -> row 1
- U1 pad 2: Net-(D2-A) -> row 2
- U1 pad 3: Net-(D3-A) -> column 1
- U1 pad 4: Net-(D4-A) -> column 2
- U1 pad 7: Net-(D5-A) -> column 3
Routing:
- net GND: track 142.6 -> 25.9 mm, vias 2 -> 0
- net Net-(D2-K): track 96.8 -> 0.00 mm
- net Net-(D1-K): track 67.8 -> 0.00 mm
- net Net-(D3-K): track 56.0 -> 0.00 mm
- net SW7 A: track 69.1 -> 122.7 mm, vias 3 -> 0
- net column 3: track 0.00 -> 50.7 mm, vias 0 -> 2
- net column 1: track 0.00 -> 46.9 mm
- net Net-(D2-A): track 9.80 -> 56.5 mm, vias 0 -> 1
- net column 2: track 0.00 -> 43.0 mm
- net Net-(D4-K): track 40.7 -> 0.00 mm, vias 1 -> 0
- net Net-(D5-K): track 38.8 -> 0.00 mm, vias 1 -> 0
- net Net-(D6-A): track 0.00 -> 31.7 mm
- net Net-(D5-A): track 9.77 -> 41.4 mm, vias 0 -> 1
- net Net-(D1-A): track 9.76 -> 39.6 mm
- net Net-(D4-A): track 9.85 -> 38.7 mm, vias 0 -> 2
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